File: eda/future_badge/future_badge.kicad_sch (KiCad schematic)
At the start: 36 parts, among them SW1 SPDT_SS12D00G, U1 ESP32-WROOM-32-DEVKIT

Commit message: incorporate updates from true
Parts:
- added C1: 10uF/50V, Capacitor_THT:C_Rect_L7.2mm_W3.5mm_P5.00mm_FKS2_FKP2_MKS2_MKP2, symbol 0_local:C_Disc_D3
- added C2, C3: 22uF/25V, 0_local:C_1206_3216Metric_Pad1.42x1.75mm_HS_Bars, symbol 0_local:C_Disc_D3
- added J1, J2, J3: Conn_01x04, 0_local:Conn_Pin_Header_Male_Vert_Back_1x04_Pitch2.54mm, symbol Connector_Generic:Conn_01x04
- added JB1, JB2, JB3: Conn_01x04, Conn_Pin_Header_Female_Vert_Back_1x04_Pitch2.54mm, symbol Connector_Generic:Conn_01x04
- added JSAO1: Addon_02x03, 0_sao_v169bis:SAOv169-BADGEv2b-PO-2x3, symbol Connector_Generic:Conn_02x03_Odd_Even
- added Q1: CJ3139K, 0_local:SOT-23_Boxed, symbol Transistor_FET:AO3401A
- added VR1: LMTOE78_0.5, 0_local:LMTOE78_0.5, symbol 0_local:LMTOE78
Connections:
- net +9V: now also SW1.3 (C), C1.1, VR1.1 (IN); no longer SW1.1 (A), U1.30 (VIN)
- net GND: now also C1.2, C2.2, C3.2, JB1.1 (Pin_1), JB1.3 (Pin_3), JB1.4 (Pin_4), JB3.2 (Pin_2), JB3.3 (Pin_3), Q1.1 (G), VR1.4 (GND)
- net TOUCH: now also JB1.2 (Pin_2); no longer TCH1.1
- net at BT1.1 (+): now also Q1.3 (D); no longer SW1.2 (B)
- net +3.3V renamed +3V3
- net +3V3: now also C2.1, C3.1, JB3.1 (Pin_1), JB3.4 (Pin_4), VR1.3 (OUT)
- new net: Q1.2 (S), SW1.2 (B)
- new net: J1.2 (Pin_2), TCH1.1
- new net 3V3_ADDON: J3.1 (Pin_1), J3.4 (Pin_4), JSAO1.1 (Pin_1)
- new net GNDFILL: J1.1 (Pin_1), J1.3 (Pin_3), J1.4 (Pin_4), J3.2 (Pin_2), J3.3 (Pin_3), JSAO1.2 (Pin_2)
- no-connect marks 12 -> 21
Other:
- note added: "Bot Board"
- note added: "Top Board"
- moved on the sheet: BT1, C11, C21, D1, D11, D2, D21, D3, D31, D32, D33, D34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
